Commit message: calibrator improvements

File: calibrator_description/urdf/calibrator.xacro (robot description, xacro)
@@ -18,12 +18,45 @@
   <link name="base_link"/>
   <link name="world" />
-  <joint name="fixed_base" type="fixed">
+  <joint name="joint_base" type="fixed">
     <parent link="world"/>
     <child link="base_link"/>
   </joint>
   <xacro:include filename="$(find calibrator_description)/urdf/checkerboard.xacro" />
-  <joint name="fixed" type="fixed">
+  <joint name="joint_fixed" type="fixed">
+    <origin xyz="0 0 0" rpy="0 0 0"/>
     <parent link="base_link"/>
+    <child link="link0"/>
+    <axis xyz="0 0 1"/>
+  </joint>
+  <link name="link0">
+    <collision>
+      <origin xyz="0 0 ${height1/2}" rpy="0 0 0"/>
+      <geometry>
+      	<box size="${width} ${width} ${height1}"/>
+      </geometry>
+    </collision>
+    <visual>
+      <origin xyz="0 0 ${height1/2}" rpy="0 0 0"/>
+      <geometry>
+      	<box size="${width} ${width} ${height1}"/>
+      </geometry>
+      <material name="orange"/>
+    </visual>
+    <inertial>
+      <origin xyz="0 0 ${height1/2}" rpy="0 0 0"/>
+      <mass value="0.1"/>
+      <inertia
+	  ixx="${mass / 12.0 * (width*width + height1*height1)}" ixy="0.0" ixz="0.0"
+	  iyy="${mass / 12.0 * (height1*height1 + width*width)}" iyz="0.0"
+	  izz="${mass / 12.0 * (width*width + width*width)}"/>
+    </inertial>
+  </link>
+  <joint name="joint0" type="prismatic">
+    <parent link="link0"/>
     <child link="link1"/>
+    <origin xyz="0 0 ${height1 - axel_offset}" rpy="0 0 0"/>
+    <axis xyz="0 0 1"/>
+    <dynamics damping="0.1"/>
+    <limit lower="-2.0" upper="0.0" effort="1000" velocity="1.0" />
   </joint>
   <!-- Base Link -->
@@ -51,10 +84,11 @@
     </inertial>
   </link>
-  <joint name="joint1" type="continuous">
+  <joint name="joint1" type="prismatic">
     <parent link="link1"/>
     <child link="link2"/>
-    <origin xyz="0 ${width} ${height1 - axel_offset}" rpy="0 0 0"/>
+    <origin xyz="${width} 0 ${height1 - axel_offset}" rpy="0 ${-pi/2} ${-pi/2}"/>
     <axis xyz="0 1 0"/>
-    <dynamics damping="0.7"/>
+    <dynamics damping="0.1"/>
+    <limit lower="-1.0" upper="1.0" effort="1.0" velocity="1.0" />
   </joint>
   <!-- Middle Link -->
@@ -85,5 +119,5 @@
     <parent link="link2"/>
     <child link="link3"/>
-    <origin xyz="0 ${width} ${height2 - axel_offset*2}" rpy="0 0 0"/>
+    <origin xyz="0 ${-width} ${height2 - axel_offset*2}" rpy="0 0 0"/>
     <axis xyz="0 1 0"/>
     <dynamics damping="0.7"/>
@@ -113,33 +147,7 @@
     </inertial>
   </link>
-  <joint name="hokuyo_joint" type="fixed">
-    <axis xyz="0 1 0" />
-    <origin xyz="0 0 ${height3 - axel_offset/2}" rpy="0 0 0"/>
-    <parent link="link3"/>
-    <child link="hokuyo_link"/>
-  </joint>
-  <!-- Hokuyo Laser -->
-  <link name="hokuyo_link">
-    <collision>
-      <origin xyz="0 0 0" rpy="0 0 0"/>
-      <geometry>
-	<box size="0.1 0.1 0.1"/>
-      </geometry>
-    </collision>
-    <visual>
-      <origin xyz="0 0 0" rpy="0 0 0"/>
-      <geometry>
-        <mesh filename="package://calibrator_description/meshes/hokuyo.dae"/>
-      </geometry>
-    </visual>
-    <inertial>
-      <mass value="1e-5" />
-      <origin xyz="0 0 0" rpy="0 0 0"/>
-      <inertia ixx="1e-6" ixy="0" ixz="0" iyy="1e-6" iyz="0" izz="1e-6" />
-    </inertial>
-  </link>
   <joint name="camera_joint" type="fixed">
     <axis xyz="0 1 0" />
-    <origin xyz="${camera_link} 0 ${height3 - axel_offset*2}" rpy="0 0 0"/>
+    <origin xyz="0 0 ${height3 - axel_offset/2}" rpy="0 ${-pi/2} ${pi}"/>
     <parent link="link3"/>
     <child link="camera_link"/>
@@ -177,4 +185,14 @@
   <link name="camera_link_optical">
   </link>
+  <transmission name="tran0">
+    <type>transmission_interface/SimpleTransmission</type>
+    <joint name="joint0">
+      <hardwareInterface>hardware_interface/EffortJointInterface</hardwareInterface>
+    </joint>
+    <actuator name="motor0">
+      <hardwareInterface>hardware_interface/EffortJointInterface</hardwareInterface>
+      <mechanicalReduction>1</mechanicalReduction>
+    </actuator>
+  </transmission>
   <transmission name="tran1">
     <type>transmission_interface/SimpleTransmission</type>

File: calibrator_description/urdf/checkerboard.xacro (robot description, xacro)
@@ -23,5 +23,5 @@
       <parent link="base_link"/>
       <child link="checkerboard_link"/>
-      <origin xyz="0 0.5 0.01" rpy="0 1.57 0" />
+      <origin xyz="0 1.0 0.01" rpy="0 1.57 1.57" />
     </joint>
 </robot>

Commit message: added the checkerboard to the world

File: calibrator_description/urdf/calibrator.xacro (robot description, xacro)
@@ -22,5 +22,5 @@
     <child link="base_link"/>
   </joint>
-  <xacro:include filename="$(find calibrator_description)/urdf/checkerboard.xacro" />
+  <!--xacro:include filename="$(find calibrator_description)/urdf/checkerboard.xacro" /-->
   <joint name="joint_fixed" type="fixed">
     <origin xyz="0 0 0" rpy="0 0 0"/>
@@ -58,12 +58,12 @@
     <axis xyz="0 0 1"/>
     <dynamics damping="0.1"/>
-    <limit lower="-2.0" upper="0.0" effort="1000" velocity="1.0" />
+    <limit lower="${-height1}" upper="0" effort="1000" velocity="1.0" />
   </joint>
   <!-- Base Link -->
   <link name="link1">
     <collision>
-      <origin xyz="0 0 ${height1/2}" rpy="0 0 0"/>
-      <geometry>
-      	<box size="${width} ${width} ${height1}"/>
+      <origin xyz="0 0 ${height1}" rpy="0 0 0"/>
+      <geometry>
+      	<box size="${width} ${width} ${height1*2}"/>
       </geometry>
     </collision>
@@ -84,11 +84,9 @@
     </inertial>
   </link>
-  <joint name="joint1" type="prismatic">
+  <joint name="joint1" type="continuous">
     <parent link="link1"/>
     <child link="link2"/>
     <origin xyz="${width} 0 ${height1 - axel_offset}" rpy="0 ${-pi/2} ${-pi/2}"/>
-    <axis xyz="0 1 0"/>
-    <dynamics damping="0.1"/>
-    <limit lower="-1.0" upper="1.0" effort="1.0" velocity="1.0" />
+    <axis xyz="0 0 1"/>
   </joint>
   <!-- Middle Link -->
@@ -119,5 +117,5 @@
     <parent link="link2"/>
     <child link="link3"/>
-    <origin xyz="0 ${-width} ${height2 - axel_offset*2}" rpy="0 0 0"/>
+    <origin xyz="0 ${-width} ${height2 - axel_offset*2}" rpy="0 ${-pi/2} 0"/>
     <axis xyz="0 1 0"/>
     <dynamics damping="0.7"/>

Commit message: working calibration

File: calibrator_description/urdf/calibrator.xacro (robot description, xacro)
@@ -16,16 +16,68 @@
   <xacro:include filename="$(find calibrator_description)/urdf/materials.xacro" />
   <!-- Used for fixing robot to Gazebo 'base_link' -->
-  <link name="base_link"/>
+  <link name="base_link">
+    <collision>
+      <origin xyz="0 0 ${width/2}" rpy="0 0 0"/>
+      <geometry>
+      	<box size="${width} ${width} ${width}"/>
+      </geometry>
+    </collision>
+    <visual>
+      <origin xyz="0 0 ${width/2}" rpy="0 0 0"/>
+      <geometry>
+      	<box size="${width} ${width} ${width}"/>
+      </geometry>
+      <material name="orange"/>
+    </visual>
+    <inertial>
+      <origin xyz="0 0 ${width/2}" rpy="0 0 0"/>
+      <mass value="${mass*1000}"/>
+      <inertia
+	  ixx="${mass / 12.0 * (width*width + width*width)}" ixy="0.0" ixz="0.0"
+	  iyy="${mass / 12.0 * (width*width + width*width)}" iyz="0.0"
+	  izz="${mass / 12.0 * (width*width + width*width)}"/>
+    </inertial>
+  </link>
   <link name="world" />
-  <joint name="joint_base" type="fixed">
+  <joint name="joint_fixed" type="fixed">
+    <origin xyz="0 0 0" rpy="0 0 0" />
     <parent link="world"/>
     <child link="base_link"/>
   </joint>
   <!--xacro:include filename="$(find calibrator_description)/urdf/checkerboard.xacro" /-->
-  <joint name="joint_fixed" type="fixed">
-    <origin xyz="0 0 0" rpy="0 0 0"/>
+  <joint name="joint_forward_backward" type="continuous">
+    <origin xyz="0 0 ${width}" rpy="0 0 0"/>
     <parent link="base_link"/>
+    <child link="link_cube"/>
+    <axis xyz="1 0 0"/>
+  </joint>
+  <link name="link_cube">
+    <collision>
+      <origin xyz="0 0 ${width/2}" rpy="0 0 0"/>
+      <geometry>
+      	<box size="${width} ${width} ${width}"/>
+      </geometry>
+    </collision>
+    <visual>
+      <origin xyz="0 0 ${width/2}" rpy="0 0 0"/>
+      <geometry>
+      	<box size="${width} ${width} ${width}"/>
+      </geometry>
+      <material name="orange"/>
+    </visual>
+    <inertial>
+      <origin xyz="0 0 ${width/2}" rpy="0 0 0"/>
+      <mass value="${mass*100}"/>
+      <inertia
+	  ixx="${mass / 12.0 * (width*width + width*width)}" ixy="0.0" ixz="0.0"
+	  iyy="${mass / 12.0 * (width*width + width*width)}" iyz="0.0"
+	  izz="${mass / 12.0 * (width*width + width*width)}"/>
+    </inertial>
+  </link>
+  <joint name="joint_left_right" type="continuous">
+    <origin xyz="0 0 ${width}" rpy="0 0 0"/>
+    <parent link="link_cube"/>
     <child link="link0"/>
-    <axis xyz="0 0 1"/>
+    <axis xyz="0 1 0"/>
   </joint>
   <link name="link0">
@@ -45,5 +97,5 @@
     <inertial>
       <origin xyz="0 0 ${height1/2}" rpy="0 0 0"/>
-      <mass value="0.1"/>
+      <mass value="${mass}"/>
       <inertia
 	  ixx="${mass / 12.0 * (width*width + height1*height1)}" ixy="0.0" ixz="0.0"
@@ -60,5 +112,4 @@
     <limit lower="${-height1}" upper="0" effort="1000" velocity="1.0" />
   </joint>
-  <!-- Base Link -->
   <link name="link1">
     <collision>
@@ -90,5 +141,4 @@
     <axis xyz="0 0 1"/>
   </joint>
-  <!-- Middle Link -->
   <link name="link2">
     <collision>
@@ -119,7 +169,5 @@
     <origin xyz="0 ${-width} ${height2 - axel_offset*2}" rpy="0 ${-pi/2} 0"/>
     <axis xyz="0 1 0"/>
-    <dynamics damping="0.7"/>
-  </joint>
-  <!-- Top Link -->
+  </joint>
   <link name="link3">
     <collision>
@@ -151,5 +199,4 @@
     <child link="camera_link"/>
   </joint>
-  <!-- Camera -->
   <link name="camera_link">
     <collision>
@@ -172,9 +219,5 @@
     </inertial>
   </link>
-  <!-- generate an optical frame http://www.ros.org/reps/rep-0103.html#suffix-frames
-      so that ros and opencv can operate on the camera frame correctly -->
   <joint name="camera_optical_joint" type="fixed">
-    <!-- these values have to be these values otherwise the gazebo camera image
-        won't be aligned properly with the frame it is supposedly originating from -->
     <origin xyz="0 0 0" rpy="${-pi/2} 0 ${-pi/2}"/>
     <parent link="camera_link"/>
@@ -183,4 +226,24 @@
   <link name="camera_link_optical">
   </link>
+  <transmission name="tran_lr">
+    <type>transmission_interface/SimpleTransmission</type>
+    <joint name="joint_left_right">
+      <hardwareInterface>hardware_interface/EffortJointInterface</hardwareInterface>
+    </joint>
+    <actuator name="motor_lr">
+      <hardwareInterface>hardware_interface/EffortJointInterface</hardwareInterface>
+      <mechanicalReduction>1</mechanicalReduction>
+    </actuator>
+  </transmission>
+  <transmission name="tran_fb">
+    <type>transmission_interface/SimpleTransmission</type>
+    <joint name="joint_forward_backward">
+      <hardwareInterface>hardware_interface/EffortJointInterface</hardwareInterface>
+    </joint>
+    <actuator name="motor_fb">
+      <hardwareInterface>hardware_interface/EffortJointInterface</hardwareInterface>
+      <mechanicalReduction>1</mechanicalReduction>
+    </actuator>
+  </transmission>
   <transmission name="tran0">
     <type>transmission_interface/SimpleTransmission</type>
